File: Eagle/ETH7820 with ESP32.sch (EAGLE design)
At the start: 40 parts

Commit message: board renew
Parts:
- removed JP1: (no value), pinhead:PINHD-1X2
- removed REFCLKO2: 33R/1%/R0603, rcl:R-EU_R0603
- added JP2: (no value), pinhead:PINHD-1X2
- added REFCLKO3: 33R/1%/R0603, rcl:R-EU_R0603
- PHY_RESET2: value no value -> do not populate
Connections:
- removed net N$12 (its old number): 2.REFCLKO/!INT, REFCLKO2.2
- removed net N$22 (its old number): REFCLKO2.1, REFCLKO4.1
- new net N$11: 2.REFCLKO/!INT, REFCLKO3.2
- new net N$21: REFCLKO3.1, REFCLKO4.1
- net +3V3: now also JP2.2; no longer JP1.2
- net GND: now also JP2.1; no longer JP1.1
Other:
- moved on the sheet: 2, C1, C11, C12, C14, C15, C16, C17, C18, C19, C20, C25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
